Commit message: orangized version of mobile_hubo sensor simulation

File: models/mobile_hubo_OW/mobile_hubo_OW.urdf (robot description, URDF)
Before this commit: robot mobile_hubo_OW, 31 links, 30 joints
Links:
- added link base_footprint
- link Body_Caster1_link: geometry collision box size=0.001 0.001 0.001; visual mesh filename=package://mobile_hubo_ow/meshes/Body_WHBASE_caster1.STL
- link Body_Caster2_link: geometry collision box size=0.001 0.001 0.001; visual mesh filename=package://mobile_hubo_ow/meshes/Body_WHBASE_caster2.STL
- link Body_Caster3_link: geometry collision box size=0.001 0.001 0.001; visual mesh filename=package://mobile_hubo_ow/meshes/Body_WHBASE_caster3.STL
- link Body_Caster4_link: geometry collision box size=0.001 0.001 0.001; visual mesh filename=package://mobile_hubo_ow/meshes/Body_WHBASE_caster4.STL
- link Body_CasterWheel1_link: geometry collision cylinder length=0.015 radius=0.025; visual mesh filename=package://mobile_hubo_ow/meshes/Body_WHBASE_casterwheel1.STL
- link Body_CasterWheel2_link: geometry collision cylinder length=0.015 radius=0.025; visual mesh filename=package://mobile_hubo_ow/meshes/Body_WHBASE_casterwheel2.STL
- link Body_CasterWheel3_link: geometry collision cylinder length=0.015 radius=0.025; visual mesh filename=package://mobile_hubo_ow/meshes/Body_WHBASE_casterwheel3.STL
- link Body_CasterWheel4_link: geometry collision cylinder length=0.015 radius=0.025; visual mesh filename=package://mobile_hubo_ow/meshes/Body_WHBASE_casterwheel4.STL
- link Body_LEB: geometry collision mesh filename=package://mobile_hubo_ow/meshes/Body_LEB_col.STL; visual mesh filename=package://mobile_hubo_ow/meshes/Body_LEB.STL
- link Body_LSP: geometry collision mesh filename=package://mobile_hubo_ow/meshes/Body_LSP_col.STL; visual mesh filename=package://mobile_hubo_ow/meshes/Body_LSP.STL
- link Body_LSR: geometry collision mesh filename=package://mobile_hubo_ow/meshes/Body_LSR_col.STL; visual mesh filename=package://mobile_hubo_ow/meshes/Body_LSR.STL
- link Body_LSY: geometry collision mesh filename=package://mobile_hubo_ow/meshes/Body_LSY_col.STL; visual mesh filename=package://mobile_hubo_ow/meshes/Body_LSY.STL
- link Body_LWFT: geometry collision mesh filename=package://mobile_hubo_ow/meshes/Body_LWFT_col.STL; visual mesh filename=package://mobile_hubo_ow/meshes/Body_LWFT.STL
- link Body_LWH_link: geometry collision cylinder length=0.03 radius=0.074; visual mesh filename=package://mobile_hubo_ow/meshes/Body_LWH_mobile.STL
- link Body_LWP: geometry collision mesh filename=package://mobile_hubo_ow/meshes/Body_LWP_col.STL; visual mesh filename=package://mobile_hubo_ow/meshes/Body_LWP.STL
- link Body_LWY: geometry collision mesh filename=package://mobile_hubo_ow/meshes/Body_LWY_col.STL; visual mesh filename=package://mobile_hubo_ow/meshes/Body_LWY.STL
- link Body_REB: geometry collision mesh filename=package://mobile_hubo_ow/meshes/Body_REB_col.STL; visual mesh filename=package://mobile_hubo_ow/meshes/Body_REB.STL
- link Body_RSP: geometry collision mesh filename=package://mobile_hubo_ow/meshes/Body_RSP_col.STL; visual mesh filename=package://mobile_hubo_ow/meshes/Body_RSP.STL
- link Body_RSR: geometry collision mesh filename=package://mobile_hubo_ow/meshes/Body_RSR_col.STL; visual mesh filename=package://mobile_hubo_ow/meshes/Body_RSR.STL
- link Body_RSY: geometry collision mesh filename=package://mobile_hubo_ow/meshes/Body_RSY_col.STL; visual mesh filename=package://mobile_hubo_ow/meshes/Body_RSY.STL
- link Body_RWFT: geometry collision mesh filename=package://mobile_hubo_ow/meshes/Body_RWFT_col.STL; visual mesh filename=package://mobile_hubo_ow/meshes/Body_RWFT.STL
- link Body_RWH_link: geometry collision cylinder length=0.03 radius=0.074; visual mesh filename=package://mobile_hubo_ow/meshes/Body_RWH_mobile.STL
- link Body_RWP: geometry collision mesh filename=package://mobile_hubo_ow/meshes/Body_RWP_col.STL; visual mesh filename=package://mobile_hubo_ow/meshes/Body_RWP.STL
- link Body_RWY: geometry collision mesh filename=package://mobile_hubo_ow/meshes/Body_RWY_col.STL; visual mesh filename=package://mobile_hubo_ow/meshes/Body_RWY.STL
- link Body_TORSO: geometry collision mesh filename=package://mobile_hubo_ow/meshes/Body_TORSO_col.STL; visual mesh filename=package://mobile_hubo_ow/meshes/Body_TORSO.STL
- link Body_WHBase_link: geometry collision box size=0.001 0.001 0.001; visual mesh filename=package://mobile_hubo_ow/meshes/Body_WHBASE.STL
- link Body_vision: geometry collision mesh filename=package://mobile_hubo_ow/meshes/ASM_VISION.STL; visual mesh filename=package://mobile_hubo_ow/meshes/ASM_VISION.STL
Joints:
- added joint base_footprint_joint: type floating, parent Body_TORSO, child base_footprint, origin xyz=0 0 0 rpy=0 0 0
