Commit message: finger added, basefootprint added, base_plate added

File: mobile_hubo_ow/urdf/mobile_hubo_OW.urdf (robot description, URDF)
Before this commit: robot mobile_hubo_OW, 27 links, 26 joints
Links:
- added link Body_LF1, mass 0.894667; collision mesh filename=package://mobile_hubo_ow/meshes/Body_LF1_col.STL; visual mesh filename=package://mobile_hubo_ow/meshes/Body_LF1.STL
- added link Body_LF2_a1, mass 0.038683; collision mesh filename=package://mobile_hubo_ow/meshes/Body_LF2_a1_col.STL; visual mesh filename=package://mobile_hubo_ow/meshes/Body_LF2_a1.STL
- added link Body_LF2_a2, mass 0.021949; collision mesh filename=package://mobile_hubo_ow/meshes/Body_LF2_a3_col.STL; visual mesh filename=package://mobile_hubo_ow/meshes/Body_LF2_a2.STL
- added link Body_LF2_a3, mass 0.0115; collision mesh filename=package://mobile_hubo_ow/meshes/Body_RF2_a3_col.STL; visual mesh filename=package://mobile_hubo_ow/meshes/Body_LF2_a3.STL
- added link Body_LF2_b1, mass 0.038683; collision mesh filename=package://mobile_hubo_ow/meshes/Body_LF2_b1_col.STL; visual mesh filename=package://mobile_hubo_ow/meshes/Body_LF2_b1.STL
- added link Body_LF2_b2, mass 0.021949; collision mesh filename=package://mobile_hubo_ow/meshes/Body_LF2_b2_col.STL; visual mesh filename=package://mobile_hubo_ow/meshes/Body_LF2_b2.STL
- added link Body_LF2_b3, mass 0.0115; collision mesh filename=package://mobile_hubo_ow/meshes/Body_LF2_b3_col.STL; visual mesh filename=package://mobile_hubo_ow/meshes/Body_LF2_b3.STL
- added link Body_LF2_c1, mass 0.038683; collision mesh filename=package://mobile_hubo_ow/meshes/Body_LF2_c1_col.STL; visual mesh filename=package://mobile_hubo_ow/meshes/Body_LF2_c1.STL
- added link Body_LF2_c2, mass 0.021949; collision mesh filename=package://mobile_hubo_ow/meshes/Body_LF2_c2_col.STL; visual mesh filename=package://mobile_hubo_ow/meshes/Body_LF2_c2.STL
- added link Body_LF2_c3, mass 0.0115; collision mesh filename=package://mobile_hubo_ow/meshes/Body_LF2_c3_col.STL; visual mesh filename=package://mobile_hubo_ow/meshes/Body_LF2_c3.STL
- added link Body_RF1, mass 0.894667; collision mesh filename=package://mobile_hubo_ow/meshes/Body_RF1_col.STL; visual mesh filename=package://mobile_hubo_ow/meshes/Body_RF1.STL
- added link Body_RF2_a1, mass 0.038683; collision mesh filename=package://mobile_hubo_ow/meshes/Body_RF2_a1_col.STL; visual mesh filename=package://mobile_hubo_ow/meshes/Body_RF2_a1.STL
- added link Body_RF2_a2, mass 0.021949; collision mesh filename=package://mobile_hubo_ow/meshes/Body_RF2_a2_col.STL; visual mesh filename=package://mobile_hubo_ow/meshes/Body_RF2_a2.STL
- added link Body_RF2_a3, mass 0.0115; collision mesh filename=package://mobile_hubo_ow/meshes/Body_RF2_a3_col.STL; visual mesh filename=package://mobile_hubo_ow/meshes/Body_RF2_a3.STL
- added link Body_RF2_b1, mass 0.038683; collision mesh filename=package://mobile_hubo_ow/meshes/Body_RF2_b1_col.STL; visual mesh filename=package://mobile_hubo_ow/meshes/Body_RF2_b1.STL
- added link Body_RF2_b2, mass 0.021949; collision mesh filename=package://mobile_hubo_ow/meshes/Body_RF2_b2_col.STL; visual mesh filename=package://mobile_hubo_ow/meshes/Body_RF2_b2.STL
- added link Body_RF2_b3, mass 0.0115; collision mesh filename=package://mobile_hubo_ow/meshes/Body_RF2_b3_col.STL; visual mesh filename=package://mobile_hubo_ow/meshes/Body_RF2_b3.STL
- added link Body_RF2_c1, mass 0.038683; collision mesh filename=package://mobile_hubo_ow/meshes/Body_RF2_c1_col.STL; visual mesh filename=package://mobile_hubo_ow/meshes/Body_RF2_c1.STL
- added link Body_RF2_c2, mass 0.021949; collision mesh filename=package://mobile_hubo_ow/meshes/Body_RF2_c2_col.STL; visual mesh filename=package://mobile_hubo_ow/meshes/Body_RF2_c2.STL
- added link Body_RF2_c3, mass 0.0115; collision mesh filename=package://mobile_hubo_ow/meshes/Body_RF2_c3_col.STL; visual mesh filename=package://mobile_hubo_ow/meshes/Body_RF2_c3.STL
- added link Body_WHBase_plate_link, mass 5.82442; collision box size=0.001 0.001 0.001; visual mesh filename=package://mobile_hubo_ow/meshes/Body_WHBASE_plate.STL
- added link Head_imu
- added link Head_realsense_camera
- added link Head_velodyne_lidar
- added link Head_zed_camera
- added link base_footprint
Joints:
- added joint Head_imu_joint: type fixed, parent Body_vision, child Head_imu, origin xyz=0 0 -0.01 rpy=0 0 0, axis 0 0 1
- added joint Head_realsense_joint: type fixed, parent Body_vision, child Head_realsense_camera, origin xyz=0.044 0 0.111 rpy=0 0.5235 0, axis 0 0 1
- added joint Head_velodyne_joint: type fixed, parent Body_vision, child Head_velodyne_lidar, origin xyz=0 0 0.036 rpy=0 0 0, axis 0 0 1
- added joint Head_zed_joint: type fixed, parent Body_vision, child Head_zed_camera, origin xyz=0.1 0 -0.028 rpy=3.14 0 0, axis 0 0 1
- added joint LHAND_a1: type revolute, parent Body_LF1, child Body_LF2_a1, origin xyz=0.02498 -0.023 -0.1471 rpy=0 0 0, axis 0 1 0, limit lower=0 upper=1.4708 effort=100000 velocity=1.0
- added joint LHAND_a2: type revolute, parent Body_LF2_a1, child Body_LF2_a2, origin xyz=0.03889 0 -0.0388 rpy=0 0.7854 0, axis 0 1 0, limit lower=0 upper=1.4708 effort=100000 velocity=1.0
- added joint LHAND_a3: type revolute, parent Body_LF2_a2, child Body_LF2_a3, origin xyz=0.04 0 0 rpy=0 0 0, axis 0 1 0, limit lower=0 upper=1.4708 effort=100000 velocity=1.0
- added joint LHAND_b1: type revolute, parent Body_LF1, child Body_LF2_b1, origin xyz=0.02498 0.0232 -0.1471 rpy=0 0 0, axis 0 1 0, limit lower=0 upper=1.4708 effort=100000 velocity=1.0
- added joint LHAND_b2: type revolute, parent Body_LF2_b1, child Body_LF2_b2, origin xyz=0.03889 0 -0.0388 rpy=0 0.7854 0, axis 0 1 0, limit lower=0 upper=1.4708 effort=100000 velocity=1.0
- added joint LHAND_b3: type revolute, parent Body_LF2_b2, child Body_LF2_b3, origin xyz=0.04 0 0 rpy=0 0 0, axis 0 1 0, limit lower=0 upper=1.4708 effort=100000 velocity=1.0
- added joint LHAND_c1: type revolute, parent Body_LF1, child Body_LF2_c1, origin xyz=-0.02502 0 -0.1471 rpy=0 0 0, axis 0 -1 0, limit lower=0 upper=1.4708 effort=100000 velocity=1.0
- added joint LHAND_c2: type revolute, parent Body_LF2_c1, child Body_LF2_c2, origin xyz=-0.03889 0 -0.0388 rpy=0 -0.7854 0, axis 0 -1 0, limit lower=0 upper=1.4708 effort=100000 velocity=1.0
- added joint LHAND_c3: type revolute, parent Body_LF2_c2, child Body_LF2_c3, origin xyz=-0.04 0 0 rpy=0 0 0, axis 0 -1 0, limit lower=0 upper=1.4708 effort=100000 velocity=1.0
- added joint LWY2: type revolute, parent Body_LWFT, child Body_LF1, origin xyz=0 0 0.0326 rpy=0 0 0, axis 0 0 1, limit lower=-5 upper=5 effort=10000000 velocity=100.0
- added joint RHAND_a1: type revolute, parent Body_RF1, child Body_RF2_a1, origin xyz=0.02498 -0.0232 -0.1471 rpy=0 0 0, axis 0 1 0, limit lower=0 upper=1.4708 effort=100000 velocity=1.0
- added joint RHAND_a2: type revolute, parent Body_RF2_a1, child Body_RF2_a2, origin xyz=0.03889 0 -0.0388 rpy=0 0.7854 0, axis 0 1 0, limit lower=0 upper=1.4708 effort=100000 velocity=1.0
- added joint RHAND_a3: type revolute, parent Body_RF2_a2, child Body_RF2_a3, origin xyz=0.04 0 0 rpy=0 0 0, axis 0 1 0, limit lower=0 upper=1.4708 effort=100000 velocity=1.0
- added joint RHAND_b1: type revolute, parent Body_RF1, child Body_RF2_b1, origin xyz=0.02498 0.023 -0.1471 rpy=0 0 0, axis 0 1 0, limit lower=0 upper=1.4708 effort=100000 velocity=1.0
- added joint RHAND_b2: type revolute, parent Body_RF2_b1, child Body_RF2_b2, origin xyz=0.03889 0 -0.0388 rpy=0 0.7854 0, axis 0 1 0, limit lower=0 upper=1.4708 effort=100000 velocity=1.0
- added joint RHAND_b3: type revolute, parent Body_RF2_b2, child Body_RF2_b3, origin xyz=0.04 0 0 rpy=0 0 0, axis 0 1 0, limit lower=0 upper=1.4708 effort=100000 velocity=1.0
- added joint RHAND_c1: type revolute, parent Body_RF1, child Body_RF2_c1, origin xyz=-0.02502 0 -0.1471 rpy=0 0 0 , axis 0 -1 0, limit lower=0 upper=1.4708 effort=100000 velocity=1.0
- added joint RHAND_c2: type revolute, parent Body_RF2_c1, child Body_RF2_c2, origin xyz=-0.03889 0 -0.0388 rpy=0 -0.7854 0, axis 0 -1 0, limit lower=0 upper=1.4708 effort=100000 velocity=1.0
- added joint RHAND_c3: type revolute, parent Body_RF2_c2, child Body_RF2_c3, origin xyz=-0.04 0 0 rpy=0 0 0, axis 0 -1 0, limit lower=0 upper=1.4708 effort=100000 velocity=1.0
- added joint RWY2: type revolute, parent Body_RWFT, child Body_RF1, origin xyz=0 0 0.0326 rpy=0 0 0, axis 0 0 1, limit lower=-5 upper=5 effort=100000 velocity=100.0
- added joint WHBASE_plate: type fixed, parent Body_WHBase_link, child Body_WHBase_plate_link, origin xyz=0 0 -0.638 rpy=0 0 0
- added joint base_footprint_joint: type floating, parent Body_TORSO, child base_footprint, origin xyz=0 0 0 rpy=0 0 0
- joint LWFT: limit lower=-5 upper=5 effort=100000 velocity=1.0 -> lower=-0 upper=0 effort=100000 velocity=1.0; type revolute -> prismatic
- joint RWFT: limit lower=-5 upper=5 effort=100000 velocity=1.0 -> lower=-0 upper=0 effort=100000 velocity=1.0; type revolute -> prismatic
- joint WHBASE: origin xyz=0 0 0 rpy=0 0 0 -> xyz=0 0 0.165 rpy=0 0 0
- joint whbase_to_caster1: origin xyz=0.2 0.08 -0.479 rpy=0 0 0 -> xyz=0.2 0.08 -0.096 rpy=0 0 0; parent Body_WHBase_link -> Body_WHBase_plate_link
- joint whbase_to_caster2: origin xyz=0.2 -0.08 -0.479 rpy=0 0 0 -> xyz=0.2 -0.08 -0.096 rpy=0 0 0; parent Body_WHBase_link -> Body_WHBase_plate_link
- joint whbase_to_caster3: origin xyz=-0.2 -0.08 -0.479 rpy=0 0 0 -> xyz=-0.2 -0.08 -0.096 rpy=0 0 0; parent Body_WHBase_link -> Body_WHBase_plate_link
- joint whbase_to_caster4: origin xyz=-0.2 0.08 -0.479 rpy=0 0 0 -> xyz=-0.2 0.08 -0.096 rpy=0 0 0; parent Body_WHBase_link -> Body_WHBase_plate_link
- joint whbase_to_lwh: origin xyz=0 0.2 -0.430 rpy=0 0 0 -> xyz=0 0.2 -0.047 rpy=0 0 0; parent Body_WHBase_link -> Body_WHBase_plate_link
- joint whbase_to_rwh: origin xyz=0 -0.2 -0.430 rpy=0 0 0 -> xyz=0 -0.2 -0.047 rpy=0 0 0; parent Body_WHBase_link -> Body_WHBase_plate_link

File: models/mobile_hubo_OW/mobile_hubo_OW.urdf (robot description, URDF)
Before this commit: robot mobile_hubo_OW, 32 links, 31 joints
Links:
- added link Body_LF1, mass 0.894667; collision mesh filename=package://mobile_hubo_ow/meshes/Body_LF1_col.STL; visual mesh filename=package://mobile_hubo_ow/meshes/Body_LF1.STL
- added link Body_LF2_a1, mass 0.038683; collision mesh filename=package://mobile_hubo_ow/meshes/Body_LF2_a1_col.STL; visual mesh filename=package://mobile_hubo_ow/meshes/Body_LF2_a1.STL
- added link Body_LF2_a2, mass 0.021949; collision mesh filename=package://mobile_hubo_ow/meshes/Body_LF2_a3_col.STL; visual mesh filename=package://mobile_hubo_ow/meshes/Body_LF2_a2.STL
- added link Body_LF2_a3, mass 0.0115; collision mesh filename=package://mobile_hubo_ow/meshes/Body_RF2_a3_col.STL; visual mesh filename=package://mobile_hubo_ow/meshes/Body_LF2_a3.STL
- added link Body_LF2_b1, mass 0.038683; collision mesh filename=package://mobile_hubo_ow/meshes/Body_LF2_b1_col.STL; visual mesh filename=package://mobile_hubo_ow/meshes/Body_LF2_b1.STL
- added link Body_LF2_b2, mass 0.021949; collision mesh filename=package://mobile_hubo_ow/meshes/Body_LF2_b2_col.STL; visual mesh filename=package://mobile_hubo_ow/meshes/Body_LF2_b2.STL
- added link Body_LF2_b3, mass 0.0115; collision mesh filename=package://mobile_hubo_ow/meshes/Body_LF2_b3_col.STL; visual mesh filename=package://mobile_hubo_ow/meshes/Body_LF2_b3.STL
- added link Body_LF2_c1, mass 0.038683; collision mesh filename=package://mobile_hubo_ow/meshes/Body_LF2_c1_col.STL; visual mesh filename=package://mobile_hubo_ow/meshes/Body_LF2_c1.STL
- added link Body_LF2_c2, mass 0.021949; collision mesh filename=package://mobile_hubo_ow/meshes/Body_LF2_c2_col.STL; visual mesh filename=package://mobile_hubo_ow/meshes/Body_LF2_c2.STL
- added link Body_LF2_c3, mass 0.0115; collision mesh filename=package://mobile_hubo_ow/meshes/Body_LF2_c3_col.STL; visual mesh filename=package://mobile_hubo_ow/meshes/Body_LF2_c3.STL
- added link Body_RF1, mass 0.894667; collision mesh filename=package://mobile_hubo_ow/meshes/Body_RF1_col.STL; visual mesh filename=package://mobile_hubo_ow/meshes/Body_RF1.STL
- added link Body_RF2_a1, mass 0.038683; collision mesh filename=package://mobile_hubo_ow/meshes/Body_RF2_a1_col.STL; visual mesh filename=package://mobile_hubo_ow/meshes/Body_RF2_a1.STL
- added link Body_RF2_a2, mass 0.021949; collision mesh filename=package://mobile_hubo_ow/meshes/Body_RF2_a2_col.STL; visual mesh filename=package://mobile_hubo_ow/meshes/Body_RF2_a2.STL
- added link Body_RF2_a3, mass 0.0115; collision mesh filename=package://mobile_hubo_ow/meshes/Body_RF2_a3_col.STL; visual mesh filename=package://mobile_hubo_ow/meshes/Body_RF2_a3.STL
- added link Body_RF2_b1, mass 0.038683; collision mesh filename=package://mobile_hubo_ow/meshes/Body_RF2_b1_col.STL; visual mesh filename=package://mobile_hubo_ow/meshes/Body_RF2_b1.STL
- added link Body_RF2_b2, mass 0.021949; collision mesh filename=package://mobile_hubo_ow/meshes/Body_RF2_b2_col.STL; visual mesh filename=package://mobile_hubo_ow/meshes/Body_RF2_b2.STL
- added link Body_RF2_b3, mass 0.0115; collision mesh filename=package://mobile_hubo_ow/meshes/Body_RF2_b3_col.STL; visual mesh filename=package://mobile_hubo_ow/meshes/Body_RF2_b3.STL
- added link Body_RF2_c1, mass 0.038683; collision mesh filename=package://mobile_hubo_ow/meshes/Body_RF2_c1_col.STL; visual mesh filename=package://mobile_hubo_ow/meshes/Body_RF2_c1.STL
- added link Body_RF2_c2, mass 0.021949; collision mesh filename=package://mobile_hubo_ow/meshes/Body_RF2_c2_col.STL; visual mesh filename=package://mobile_hubo_ow/meshes/Body_RF2_c2.STL
- added link Body_RF2_c3, mass 0.0115; collision mesh filename=package://mobile_hubo_ow/meshes/Body_RF2_c3_col.STL; visual mesh filename=package://mobile_hubo_ow/meshes/Body_RF2_c3.STL
- added link Body_WHBase_plate_link, mass 5.82442; collision box size=0.001 0.001 0.001; visual mesh filename=package://mobile_hubo_ow/meshes/Body_WHBASE_plate.STL
Joints:
- added joint LHAND_a1: type revolute, parent Body_LF1, child Body_LF2_a1, origin xyz=0.02498 -0.023 -0.1471 rpy=0 0 0, axis 0 1 0, limit lower=0 upper=1.4708 effort=100000 velocity=1.0
- added joint LHAND_a2: type revolute, parent Body_LF2_a1, child Body_LF2_a2, origin xyz=0.03889 0 -0.0388 rpy=0 0.7854 0, axis 0 1 0, limit lower=0 upper=1.4708 effort=100000 velocity=1.0
- added joint LHAND_a3: type revolute, parent Body_LF2_a2, child Body_LF2_a3, origin xyz=0.04 0 0 rpy=0 0 0, axis 0 1 0, limit lower=0 upper=1.4708 effort=100000 velocity=1.0
- added joint LHAND_b1: type revolute, parent Body_LF1, child Body_LF2_b1, origin xyz=0.02498 0.0232 -0.1471 rpy=0 0 0, axis 0 1 0, limit lower=0 upper=1.4708 effort=100000 velocity=1.0
- added joint LHAND_b2: type revolute, parent Body_LF2_b1, child Body_LF2_b2, origin xyz=0.03889 0 -0.0388 rpy=0 0.7854 0, axis 0 1 0, limit lower=0 upper=1.4708 effort=100000 velocity=1.0
- added joint LHAND_b3: type revolute, parent Body_LF2_b2, child Body_LF2_b3, origin xyz=0.04 0 0 rpy=0 0 0, axis 0 1 0, limit lower=0 upper=1.4708 effort=100000 velocity=1.0
- added joint LHAND_c1: type revolute, parent Body_LF1, child Body_LF2_c1, origin xyz=-0.02502 0 -0.1471 rpy=0 0 0, axis 0 -1 0, limit lower=0 upper=1.4708 effort=100000 velocity=1.0
- added joint LHAND_c2: type revolute, parent Body_LF2_c1, child Body_LF2_c2, origin xyz=-0.03889 0 -0.0388 rpy=0 -0.7854 0, axis 0 -1 0, limit lower=0 upper=1.4708 effort=100000 velocity=1.0
- added joint LHAND_c3: type revolute, parent Body_LF2_c2, child Body_LF2_c3, origin xyz=-0.04 0 0 rpy=0 0 0, axis 0 -1 0, limit lower=0 upper=1.4708 effort=100000 velocity=1.0
- added joint LWY2: type revolute, parent Body_LWFT, child Body_LF1, origin xyz=0 0 0.0326 rpy=0 0 0, axis 0 0 1, limit lower=-5 upper=5 effort=10000000 velocity=100.0
- added joint RHAND_a1: type revolute, parent Body_RF1, child Body_RF2_a1, origin xyz=0.02498 -0.0232 -0.1471 rpy=0 0 0, axis 0 1 0, limit lower=0 upper=1.4708 effort=100000 velocity=1.0
- added joint RHAND_a2: type revolute, parent Body_RF2_a1, child Body_RF2_a2, origin xyz=0.03889 0 -0.0388 rpy=0 0.7854 0, axis 0 1 0, limit lower=0 upper=1.4708 effort=100000 velocity=1.0
- added joint RHAND_a3: type revolute, parent Body_RF2_a2, child Body_RF2_a3, origin xyz=0.04 0 0 rpy=0 0 0, axis 0 1 0, limit lower=0 upper=1.4708 effort=100000 velocity=1.0
- added joint RHAND_b1: type revolute, parent Body_RF1, child Body_RF2_b1, origin xyz=0.02498 0.023 -0.1471 rpy=0 0 0, axis 0 1 0, limit lower=0 upper=1.4708 effort=100000 velocity=1.0
- added joint RHAND_b2: type revolute, parent Body_RF2_b1, child Body_RF2_b2, origin xyz=0.03889 0 -0.0388 rpy=0 0.7854 0, axis 0 1 0, limit lower=0 upper=1.4708 effort=100000 velocity=1.0
- added joint RHAND_b3: type revolute, parent Body_RF2_b2, child Body_RF2_b3, origin xyz=0.04 0 0 rpy=0 0 0, axis 0 1 0, limit lower=0 upper=1.4708 effort=100000 velocity=1.0
- added joint RHAND_c1: type revolute, parent Body_RF1, child Body_RF2_c1, origin xyz=-0.02502 0 -0.1471 rpy=0 0 0 , axis 0 -1 0, limit lower=0 upper=1.4708 effort=100000 velocity=1.0
- added joint RHAND_c2: type revolute, parent Body_RF2_c1, child Body_RF2_c2, origin xyz=-0.03889 0 -0.0388 rpy=0 -0.7854 0, axis 0 -1 0, limit lower=0 upper=1.4708 effort=100000 velocity=1.0
- added joint RHAND_c3: type revolute, parent Body_RF2_c2, child Body_RF2_c3, origin xyz=-0.04 0 0 rpy=0 0 0, axis 0 -1 0, limit lower=0 upper=1.4708 effort=100000 velocity=1.0
- added joint RWY2: type revolute, parent Body_RWFT, child Body_RF1, origin xyz=0 0 0.0326 rpy=0 0 0, axis 0 0 1, limit lower=-5 upper=5 effort=100000 velocity=100.0
- added joint WHBASE_plate: type fixed, parent Body_WHBase_link, child Body_WHBase_plate_link, origin xyz=0 0 -0.638 rpy=0 0 0
- joint LWFT: limit lower=-5 upper=5 effort=100000 velocity=1.0 -> lower=-0 upper=0 effort=100000 velocity=1.0; type revolute -> prismatic
- joint RWFT: limit lower=-5 upper=5 effort=100000 velocity=1.0 -> lower=-0 upper=0 effort=100000 velocity=1.0; type revolute -> prismatic
- joint WHBASE: origin xyz=0 0 0 rpy=0 0 0 -> xyz=0 0 0.165 rpy=0 0 0
- joint whbase_to_caster1: origin xyz=0.2 0.08 -0.479 rpy=0 0 0 -> xyz=0.2 0.08 -0.096 rpy=0 0 0; parent Body_WHBase_link -> Body_WHBase_plate_link
- joint whbase_to_caster2: origin xyz=0.2 -0.08 -0.479 rpy=0 0 0 -> xyz=0.2 -0.08 -0.096 rpy=0 0 0; parent Body_WHBase_link -> Body_WHBase_plate_link
- joint whbase_to_caster3: origin xyz=-0.2 -0.08 -0.479 rpy=0 0 0 -> xyz=-0.2 -0.08 -0.096 rpy=0 0 0; parent Body_WHBase_link -> Body_WHBase_plate_link
- joint whbase_to_caster4: origin xyz=-0.2 0.08 -0.479 rpy=0 0 0 -> xyz=-0.2 0.08 -0.096 rpy=0 0 0; parent Body_WHBase_link -> Body_WHBase_plate_link
- joint whbase_to_lwh: origin xyz=0 0.2 -0.430 rpy=0 0 0 -> xyz=0 0.2 -0.047 rpy=0 0 0; parent Body_WHBase_link -> Body_WHBase_plate_link
- joint whbase_to_rwh: origin xyz=0 -0.2 -0.430 rpy=0 0 0 -> xyz=0 -0.2 -0.047 rpy=0 0 0; parent Body_WHBase_link -> Body_WHBase_plate_link

Commit message: rviz fixed

File: mobile_hubo_ow/urdf/mobile_hubo_OW.urdf (robot description, URDF)
Before this commit: robot mobile_hubo_OW, 53 links, 52 joints
Joints:
- joint base_footprint_joint: child base_footprint -> Body_TORSO; parent Body_TORSO -> base_footprint

Commit message: correcting changes

File: mobile_hubo_ow/urdf/mobile_hubo_OW.urdf (robot description, URDF)
Before this commit: robot mobile_hubo_OW, 53 links, 52 joints
Joints:
- joint base_footprint_joint: child Body_TORSO -> base_footprint; parent base_footprint -> Body_TORSO
